Commit message: feat: Add joint and link to xacro

File: catkin_ws/src/my_robot/urdf/my_robot.xacro (robot description, xacro)
@@ -33,4 +33,11 @@
     </visual>
   </link>
+  <joint name="camera_optical_joint" type="fixed">
+    <origin xyz="0 0 0" rpy="-1.5707 0 -1.5707"/>
+    <parent link="camera"/>
+    <child link="camera_link_optical"/>
+  </joint>
+  <link name="camera_link_optical">
+  </link>
   <link name="hokuyo">
     <pose>0 0 0 0 0 0</pose>

Commit message: fix: Add hokuyo counterbalance in the back
I'm trying to fix the car toppling forward on stop problem. I don't
think I'll be able to get rid of the problem completely. But I'm just
going to add things till it kinda sorta does not topple.

This may require that the car never speed up very much. I guess that is
okay for now.

File: catkin_ws/src/my_robot/urdf/my_robot.xacro (robot description, xacro)
@@ -64,4 +64,22 @@
     </visual>
   </link>
+  <link name="hokuyo_counter">
+    <pose>0 0 0 0 0 0</pose>
+    <inertial>
+      <mass value="1e-5"/>
+      <origin xyz="0 0 0" rpy="0 0 0"/>
+      <inertia
+          ixx="1e-6" ixy="0" ixz="0"
+          iyy="1e-6" iyz="0"
+          izz="1e-6"
+      />
+    </inertial>
+    <collision>
+      <origin xyz="0 0 0" rpy="0 0 0"/>
+      <geometry>
+        <box size="0.1 0.1 0.1"/>
+      </geometry>
+    </collision>
+  </link>
   <link name="left_wheel">
     <inertial>
@@ -204,4 +222,10 @@
     <child link="hokuyo" />
   </joint>
+  <joint name="hokuyo_counter_joint" type="fixed">
+    <origin xyz="-0.15 0 0.15" rpy="0 0 0" />
+    <axis xyz="0 1 0" rpy="0 0 0"/>
+    <parent link="chassis"/>
+    <child link="hokuyo_counter" />
+  </joint>
   <joint name="spoiler_joint" type="fixed">
     <origin xyz="-0.4 0 0" rpy="0 0 0" />

Commit message: fix: Stick casters out more, make frictionless
This is another attempt to reduce the toppling behaviour.

File: catkin_ws/src/my_robot/urdf/my_robot.xacro (robot description, xacro)
@@ -170,11 +170,21 @@
     </visual>
     <collision name='back_caster_collision'>
-      <origin xyz="-0.25 0 -0.1" rpy=" 0 0 0"/>
+      <origin xyz="-0.3 0 -0.1" rpy=" 0 0 0"/>
       <geometry>
         <sphere radius="0.099"/>
       </geometry>
+      <surface>
+        <friction>
+          <ode>
+            <mu>0</mu>
+            <mu2>0</mu2>
+            <slip1>1.0</slip1>
+            <slip2>1.0</slip2>
+          </ode>
+        </friction>
+      </surface>
     </collision>
     <!-- <visual name='back_caster_visual'>
-      <origin xyz="-0.25 0 -0.1" rpy=" 0 0 0"/>
+      <origin xyz="-0.3 0 -0.1" rpy=" 0 0 0"/>
       <geometry>
         <sphere radius="0.1"/>
@@ -182,11 +192,21 @@
     </visual> -->
     <collision name='front_caster_collision'>
-      <origin xyz="0.25 0 -0.1" rpy=" 0 0 0"/>
+      <origin xyz="0.3 0 -0.1" rpy=" 0 0 0"/>
       <geometry>
         <sphere radius="0.099"/>
       </geometry>
+      <surface>
+        <friction>
+          <ode>
+            <mu>0</mu>
+            <mu2>0</mu2>
+            <slip1>1.0</slip1>
+            <slip2>1.0</slip2>
+          </ode>
+        </friction>
+      </surface>
     </collision>
     <!-- <visual name='front_caster_visual'>
-      <origin xyz="0.25 0 -0.1" rpy=" 0 0 0"/>
+      <origin xyz="0.3 0 -0.1" rpy=" 0 0 0"/>
       <geometry>
         <sphere radius="0.1"/>
